Commit message: First thymio bqsic design done and working with gazebo

File: src/ros_basics_2019/urdf/robot_description.urdf (robot description, URDF)
Before this commit: robot BOBBY, 16 links, 15 joints
Links:
- removed link box
- removed link gripper_pole
- removed link head
- removed link left_back_wheel
- removed link left_base
- removed link left_front_wheel
- removed link left_gripper
- removed link left_tip
- removed link right_back_wheel
- removed link right_base
- removed link right_front_wheel
- removed link right_gripper
- removed link right_tip
- added link sphere; collision sphere radius=0.05; visual sphere radius=0.1
- link base_link: mass None -> 10; geometry collision box size=0.6 0.6 0.2; visual box size=0.6 0.6 0.2
- link left_leg: geometry collision cylinder length=0.2 radius=0.15; visual cylinder length=0.2 radius=0.15
- link right_leg: geometry collision cylinder length=0.2 radius=0.15; visual cylinder length=0.2 radius=0.15
Joints:
- removed joint gripper_extension
- removed joint head_swivel
- removed joint left_back_wheel_joint
- removed joint left_base_joint
- removed joint left_front_wheel_joint
- removed joint left_gripper_joint
- removed joint left_tip_joint
- removed joint right_back_wheel_joint
- removed joint right_base_joint
- removed joint right_front_wheel_joint
- removed joint right_gripper_joint
- removed joint right_tip_joint
- removed joint tobox
- added joint base_to_sphere: type fixed, parent base_link, child sphere, origin xyz=0 -0.22 -0.10
- joint base_to_left_leg: origin xyz=0 0.22 0.25 -> xyz=-0.2 0.22 0.30
- joint base_to_right_leg: origin xyz=0 -0.22 0.25 -> xyz=0.2 0.22 0.30

File: src/ros_basics_2019/urdf/robot_description.urdf.xacro (robot description, xacro)
@@ -1,221 +1,120 @@
 <?xml version="1.0"?>
-<robot xmlns:xacro="https://www.ros.org/wiki/xacro" name="BOBBY">
+<robot xmlns:xacro="https://www.ros.org/wiki/xacro" name="YOUR_ROBOT_NAME">
+    <xacro:include filename="$(find ros_basics_2019)/urdf/macros.xacro" />
+    <xacro:include filename="$(find ros_basics_2019)/urdf/materials.xacro" />
     <!-- Design your robot here -->
-<material name="blue">
-    <color rgba="0 0 0.8 1"/>
-  </material>
-  <material name="black">
-    <color rgba="0 0 0 1"/>
-  </material>
-  <material name="white">
-    <color rgba="1 1 1 1"/>
-  </material>
   <link name="base_link">
-    <visual>
-      <geometry>
-        <cylinder length="0.6" radius="0.2"/>
-      </geometry>
-      <material name="blue"/>
-    </visual>
-  </link>
+	<visual>
+		<geometry>
+        <box size="0.6 0.6 0.2"/>
+		</geometry>
+	</visual>
+	<collision>
+	      <geometry>
+        <box size="0.6 0.6 0.2"/>
+	      </geometry>
+	</collision>
+     <inertial>
+       <mass value="10"/>
+       <inertia ixx="0.4" ixy="0.0" ixz="0.0" iyy="0.4" iyz="0.0" izz="0.2"/>
+     </inertial>
+</link>
   <link name="right_leg">
     <visual>
       <geometry>
-        <box size="0.6 0.1 0.2"/>
+		<cylinder length="0.2" radius="0.15"/>
       </geometry>
       <origin rpy="0 1.57075 0" xyz="0 0 -0.3"/>
-      <material name="white"/>
     </visual>
+<collision>
+      <geometry>
+		<cylinder length="0.2" radius="0.15"/>
+      </geometry>
+</collision>
   </link>
   <joint name="base_to_right_leg" type="fixed">
     <parent link="base_link"/>
     <child link="right_leg"/>
-    <origin xyz="0 -0.22 0.25"/>
-  </joint>
-  <link name="right_base">
-    <visual>
-      <geometry>
-        <box size="0.4 0.1 0.1"/>
-      </geometry>
-      <material name="white"/>
-    </visual>
-  </link>
-  <joint name="right_base_joint" type="fixed">
-    <parent link="right_leg"/>
-    <child link="right_base"/>
-    <origin xyz="0 0 -0.6"/>
-  </joint>
-  <link name="right_front_wheel">
-    <visual>
-      <origin rpy="1.57075 0 0" xyz="0 0 0"/>
-      <geometry>
-        <cylinder length="0.1" radius="0.035"/>
-      </geometry>
-      <material name="black"/>
-      <origin rpy="0 0 0" xyz="0 0 0"/>
-    </visual>
-  </link>
-  <joint name="right_front_wheel_joint" type="fixed">
-    <parent link="right_base"/>
-    <child link="right_front_wheel"/>
-    <origin rpy="0 0 0" xyz="0.133333333333 0 -0.085"/>
-  </joint>
-  <link name="right_back_wheel">
-    <visual>
-      <origin rpy="1.57075 0 0" xyz="0 0 0"/>
-      <geometry>
-        <cylinder length="0.1" radius="0.035"/>
-      </geometry>
-      <material name="black"/>
-    </visual>
-  </link>
-  <joint name="right_back_wheel_joint" type="fixed">
-    <parent link="right_base"/>
-    <child link="right_back_wheel"/>
-    <origin rpy="0 0 0" xyz="-0.133333333333 0 -0.085"/>
+    <origin xyz="0.2 0.22 0.30"/>
   </joint>
   <link name="left_leg">
     <visual>
       <geometry>
-        <box size="0.6 0.1 0.2"/>
+		<cylinder length="0.2" radius="0.15"/>
       </geometry>
       <origin rpy="0 1.57075 0" xyz="0 0 -0.3"/>
-      <material name="white"/>
     </visual>
+<collision>
+      <geometry>
+		<cylinder length="0.2" radius="0.15"/>
+      </geometry>
+</collision>
   </link>
   <joint name="base_to_left_leg" type="fixed">
     <parent link="base_link"/>
     <child link="left_leg"/>
-    <origin xyz="0 0.22 0.25"/>
+    <origin xyz="-0.2 0.22 0.30"/>
   </joint>
-  <link name="left_base">
+  <link name="sphere">
     <visual>
       <geometry>
-        <box size="0.4 0.1 0.1"/>
-      </geometry>
-      <material name="white"/>
-    </visual>
-  </link>
-  <joint name="left_base_joint" type="fixed">
-    <parent link="left_leg"/>
-    <child link="left_base"/>
-    <origin xyz="0 0 -0.6"/>
-  </joint>
-  <link name="left_front_wheel">
-    <visual>
-      <origin rpy="1.57075 0 0" xyz="0 0 0"/>
-      <geometry>
-        <cylinder length="0.1" radius="0.035"/>
-      </geometry>
-      <material name="black"/>
-    </visual>
-  </link>
-  <joint name="left_front_wheel_joint" type="fixed">
-    <parent link="left_base"/>
-    <child link="left_front_wheel"/>
-    <origin rpy="0 0 0" xyz="0.133333333333 0 -0.085"/>
-  </joint>
-  <link name="left_back_wheel">
-    <visual>
-      <origin rpy="1.57075 0 0" xyz="0 0 0"/>
-      <geometry>
-        <cylinder length="0.1" radius="0.035"/>
-      </geometry>
-      <material name="black"/>
-    </visual>
-  </link>
-  <joint name="left_back_wheel_joint" type="fixed">
-    <parent link="left_base"/>
-    <child link="left_back_wheel"/>
-    <origin rpy="0 0 0" xyz="-0.133333333333 0 -0.085"/>
-  </joint>
-  <joint name="gripper_extension" type="fixed">
-    <parent link="base_link"/>
-    <child link="gripper_pole"/>
-    <origin rpy="0 0 0" xyz="0.19 0 0.2"/>
-  </joint>
-  <link name="gripper_pole">
-    <visual>
-      <geometry>
-        <cylinder length="0.2" radius="0.01"/>
-      </geometry>
-      <origin rpy="0 1.57075 0 " xyz="0.1 0 0"/>
-    </visual>
-  </link>
-  <joint name="left_gripper_joint" type="fixed">
-    <origin rpy="0 0 0" xyz="0.2 0.01 0"/>
-    <parent link="gripper_pole"/>
-    <child link="left_gripper"/>
-  </joint>
-  <link name="left_gripper">
-    <visual>
-      <origin rpy="0.0 0 0" xyz="0 0 0"/>
-      <geometry>
-        <mesh filename="package://urdf_tutorial/meshes/l_finger.dae"/>
+        <sphere radius="0.1"/>
       </geometry>
     </visual>
+<collision>
+      <geometry>
+        <sphere radius="0.05"/>
+      </geometry>
+</collision>
   </link>
-  <joint name="left_tip_joint" type="fixed">
-    <parent link="left_gripper"/>
-    <child link="left_tip"/>
+  <joint name="base_to_sphere" type="fixed">
+    <parent link="base_link"/>
+    <child link="sphere"/>
+    <origin xyz="0 -0.22 -0.10"/>
   </joint>
-  <link name="left_tip">
-    <visual>
-      <origin rpy="0.0 0 0" xyz="0.09137 0.00495 0"/>
-      <geometry>
-        <mesh filename="package://urdf_tutorial/meshes/l_finger_tip.dae"/>
-      </geometry>
-    </visual>
-  </link>
-  <joint name="right_gripper_joint" type="fixed">
-    <origin rpy="0 0 0" xyz="0.2 -0.01 0"/>
-    <parent link="gripper_pole"/>
-    <child link="right_gripper"/>
-  </joint>
-  <link name="right_gripper">
-    <visual>
-      <origin rpy="-3.1415 0 0" xyz="0 0 0"/>
-      <geometry>
-        <mesh filename="package://urdf_tutorial/meshes/l_finger.dae"/>
-      </geometry>
-    </visual>
-  </link>
-  <joint name="right_tip_joint" type="fixed">
-    <parent link="right_gripper"/>
-    <child link="right_tip"/>
-  </joint>
-  <link name="right_tip">
-    <visual>
-      <origin rpy="-3.1415 0 0" xyz="0.09137 0.00495 0"/>
-      <geometry>
-        <mesh filename="package://urdf_tutorial/meshes/l_finger_tip.dae"/>
-      </geometry>
-    </visual>
-  </link>
-  <link name="head">
-    <visual>
-      <geometry>
-        <sphere radius="0.2"/>
-      </geometry>
-      <material name="white"/>
-    </visual>
-  </link>
-  <joint name="head_swivel" type="fixed">
-    <parent link="base_link"/>
-    <child link="head"/>
-    <origin xyz="0 0 0.3"/>
-  </joint>
-  <link name="box">
-    <visual>
-      <geometry>
-        <box size="0.08 0.08 0.08"/>
-      </geometry>
-      <material name="blue"/>
-    </visual>
-  </link>
-  <joint name="tobox" type="fixed">
-    <parent link="head"/>
-    <child link="box"/>
-    <origin xyz="0.1814 0 0.1414"/>
-  </joint>
+    <!-- Below you will find samples of gazebo plugins you may want to use. -->
+    <!-- These should be adapted to your robot's design -->
+    <gazebo reference="YOUR_SENSOR_LINK">
+        <sensor type="ray" name="laser_right">
+            <pose>0 0 0 0 0 0</pose>
+            <ray>
+                <scan>
+                    <horizontal>
+                        <samples>13</samples>
+                        <resolution>1</resolution>
+                        <min_angle>-1.571</min_angle>
+                        <max_angle>1.571</max_angle>
+                    </horizontal>
+                </scan>
+                <range>
+                    <!-- You can edit adapt these to your robot's size -->
+                    <min>0.0005</min>
+                    <max>0.04</max>
+                    <resolution>0.0001</resolution>
+                </range>
+            </ray>
+            <plugin name="laser" filename="libgazebo_ros_laser.so" >
+                <topicName>YOUR_ROBOT_LASER/scan</topicName>
+                <frameName>YOUR_ROBOT_LASER_LINK</frameName>
+            </plugin>
+            <always_on>1</always_on>
+            <update_rate>10</update_rate>
+            <visualize>true</visualize>
+        </sensor>
+    </gazebo>
+    <gazebo>
+        <plugin name="differential_drive_controller" filename="libgazebo_ros_diff_drive.so">
+            <alwaysOn>true</alwaysOn>
+            <updateRate>20</updateRate>
+            <leftJoint>YOUR_LEFT_WHEEL_JOINT</leftJoint>
+            <rightJoint>YOUR_RIGHT_WHEEL_JOINT</rightJoint>
+            <wheelSeparation>XXX</wheelSeparation>
+            <wheelDiameter>YYY</wheelDiameter>
+            <wheelTorque>ZZZ</wheelTorque>
+            <commandTopic>cmd_vel</commandTopic>
+            <odometryTopic>odom</odometryTopic>
+            <odometryFrame>odom</odometryFrame>
+            <robotBaseFrame>YOUR_BASE_FRAME</robotBaseFrame>
+        </plugin>
+    </gazebo>
 </robot>

Commit message: right joint for wheels

File: src/ros_basics_2019/urdf/robot_description.urdf (robot description, URDF)
Before this commit: robot YOUR_ROBOT_NAME, 4 links, 3 joints
Links:
- link left_leg: mass None -> 1; geometry collision cylinder length=0.2 radius=0.1; visual cylinder length=0.2 radius=0.1
- link right_leg: mass None -> 1; geometry collision cylinder length=0.2 radius=0.1; visual cylinder length=0.2 radius=0.1
- link sphere: mass None -> 1; geometry collision sphere radius=0.1; visual sphere radius=0.1
Joints:
- joint base_to_left_leg: axis (none) -> 1 0 0; type fixed -> continuous
- joint base_to_right_leg: axis (none) -> 1 0 0; type fixed -> continuous
- joint base_to_sphere: origin xyz=0 -0.22 -0.10 -> xyz=0 -0.22 -0.02

File: src/ros_basics_2019/urdf/robot_description.urdf.xacro (robot description, xacro)
@@ -1,4 +1,4 @@
 <?xml version="1.0"?>
-<robot xmlns:xacro="https://www.ros.org/wiki/xacro" name="YOUR_ROBOT_NAME">
+<robot xmlns:xacro="https://www.ros.org/wiki/xacro" name="BOBBY">
     <xacro:include filename="$(find ros_basics_2019)/urdf/macros.xacro" />
     <xacro:include filename="$(find ros_basics_2019)/urdf/materials.xacro" />
@@ -9,8 +9,9 @@
         <box size="0.6 0.6 0.2"/>
 		</geometry>
+		<origin xyz="0 0 +0.05"/>
 	</visual>
 	<collision>
 	      <geometry>
-        <box size="0.6 0.6 0.2"/>
+	  <box size="0.6 0.6 0.2"/>
 	      </geometry>
 	</collision>
@@ -23,36 +24,46 @@
     <visual>
       <geometry>
-		<cylinder length="0.2" radius="0.15"/>
+		<cylinder length="0.2" radius="0.1"/>
       </geometry>
-      <origin rpy="0 1.57075 0" xyz="0 0 -0.3"/>
+      <origin rpy="0 1.57075 0" xyz="0 0 0"/>
     </visual>
 <collision>
       <geometry>
-		<cylinder length="0.2" radius="0.15"/>
+		<cylinder length="0.2" radius="0.1"/>
       </geometry>
 </collision>
+     <inertial>
+       <mass value="1"/>
+       <inertia ixx="0.4" ixy="0.0" ixz="0.0" iyy="1.57" iyz="0.0" izz="0.2"/>
+     </inertial>
   </link>
-  <joint name="base_to_right_leg" type="fixed">
+  <joint name="base_to_right_leg" type="continuous">
+	<axis xyz= "1 0 0"/>
     <parent link="base_link"/>
     <child link="right_leg"/>
-    <origin xyz="0.2 0.22 0.30"/>
+    <origin xyz="0.2 0.22 0.00"/>
   </joint>
   <link name="left_leg">
     <visual>
       <geometry>
-		<cylinder length="0.2" radius="0.15"/>
+		<cylinder length="0.2" radius="0.1"/>
       </geometry>
-      <origin rpy="0 1.57075 0" xyz="0 0 -0.3"/>
+      <origin rpy="0 1.57075 0" xyz="0 0 0"/>
     </visual>
 <collision>
       <geometry>
-		<cylinder length="0.2" radius="0.15"/>
+		<cylinder length="0.2" radius="0.1"/>
       </geometry>
 </collision>
+     <inertial>
+       <mass value="1"/>
+       <inertia ixx="0.4" ixy="0.0" ixz="0.0" iyy="1.57" iyz="0.0" izz="0.2"/>
+     </inertial>
   </link>
-  <joint name="base_to_left_leg" type="fixed">
+  <joint name="base_to_left_leg" type="continuous">
     <parent link="base_link"/>
     <child link="left_leg"/>
-    <origin xyz="-0.2 0.22 0.30"/>
+	<axis xyz= "1 0 0"/>
+    <origin xyz="-0.2 0.22 0.00"/>
   </joint>
   <link name="sphere">
@@ -64,12 +75,16 @@
 <collision>
       <geometry>
-        <sphere radius="0.05"/>
+        <sphere radius="0.1"/>
       </geometry>
 </collision>
+     <inertial>
+       <mass value="1"/>
+       <inertia ixx="0.4" ixy="0.0" ixz="0.0" iyy="0.4" iyz="0.0" izz="0.2"/>
+     </inertial>
   </link>
   <joint name="base_to_sphere" type="fixed">
     <parent link="base_link"/>
     <child link="sphere"/>
-    <origin xyz="0 -0.22 -0.10"/>
+    <origin xyz="0 -0.22 -0.02"/>
   </joint>
     <!-- Below you will find samples of gazebo plugins you may want to use. -->
@@ -107,13 +122,13 @@
             <alwaysOn>true</alwaysOn>
             <updateRate>20</updateRate>
-            <leftJoint>YOUR_LEFT_WHEEL_JOINT</leftJoint>
-            <rightJoint>YOUR_RIGHT_WHEEL_JOINT</rightJoint>
-            <wheelSeparation>XXX</wheelSeparation>
-            <wheelDiameter>YYY</wheelDiameter>
+            <leftJoint>base_to_left_leg</leftJoint>
+            <rightJoint>base_to_right_leg</rightJoint>
+            <wheelSeparation>0.6</wheelSeparation>
+            <wheelDiameter>0.2</wheelDiameter>
             <wheelTorque>ZZZ</wheelTorque>
             <commandTopic>cmd_vel</commandTopic>
             <odometryTopic>odom</odometryTopic>
             <odometryFrame>odom</odometryFrame>
-            <robotBaseFrame>YOUR_BASE_FRAME</robotBaseFrame>
+            <robotBaseFrame>base_link</robotBaseFrame>
         </plugin>
     </gazebo>

Commit message: Basic robot design moving and publisher/listener nodes working with hello world

File: src/ros_basics_2019/urdf/robot_description.urdf (robot description, URDF)
Before this commit: robot BOBBY, 4 links, 3 joints
Joints:
- joint base_to_left_leg: origin xyz=-0.2 0.22 0.30 -> xyz=-0.2 0.22 0.00
- joint base_to_right_leg: origin xyz=0.2 0.22 0.30 -> xyz=0.2 0.22 0.00
- joint base_to_sphere: axis (none) -> 1 0 0; type fixed -> continuous

File: src/ros_basics_2019/urdf/robot_description.urdf.xacro (robot description, xacro)
@@ -83,7 +83,8 @@
      </inertial>
   </link>
-  <joint name="base_to_sphere" type="fixed">
+  <joint name="base_to_sphere" type="continuous">
     <parent link="base_link"/>
     <child link="sphere"/>
+<axis xyz= "1 0 0"/>
     <origin xyz="0 -0.22 -0.02"/>
   </joint>
@@ -126,5 +127,5 @@
             <wheelSeparation>0.6</wheelSeparation>
             <wheelDiameter>0.2</wheelDiameter>
-            <wheelTorque>ZZZ</wheelTorque>
+            <wheelTorque>20</wheelTorque>
             <commandTopic>cmd_vel</commandTopic>
             <odometryTopic>odom</odometryTopic>
